File: pendrive pcb/board.sch (KiCad schematic (older format))
At the start: 21 parts, among them J1 Conn_01x03_Male, J2 Conn_01x03_Male, J3 USB_A, SW1 SW_Push, SW2 SW_Push, SW3 SW_SPST, U1 PIC18F2550-ISP, Y1 8Mhz

Commit message: Switch moved to top
Parts:
- SW3: footprint Board:switch -> Button_Switch_SMD:SW_SPST_EVQPE1
